Commit message: Changed mu1, mu2 and kd

File: urdf/macros.xacro (robot description, xacro)
@@ -25,8 +25,8 @@
     </joint>
     <gazebo reference="${lr}_wheel">
-      <mu1 value="200"/>
-      <mu2 value="100"/>
+      <mu1 value="0.7"/>
+      <mu2 value="0.5"/>
       <kp value="10000000.0"/>
-      <kd value="1.0"/>
+      <kd value="100.0"/>
       <!-- <! <fdir1 value="1 0 0"/> -> -->
       <material>Gazebo/Black</material>
@@ -48,11 +48,5 @@
     </inertial>
   </xacro:macro>
-  <xacro:macro name="cylinder_inertia" params="m r h">
-    <inertia ixx="${m*(3*r*r+h*h)/12}" ixy="0" ixz="0" iyy="${m*(3*r*r+h*h)/12}" iyz="0" izz="${m*r*r/2}"/>
-  </xacro:macro>
-  <xacro:macro name="box_inertia" params="m x y z">
-    <inertia ixx="${m*(y*y+z*z)/12}" ixy="0" ixz="0" iyy="${m*(x*x+z*z)/12}" iyz="0" izz="${m*(x*x+z*z)/12}"/>
-  </xacro:macro>
-  <xacro:macro name="sphere_inertia" params="m r">
+  <xacro:macro name="cylinder_inertwheelMass" params="m r">
     <inertia ixx="${2*m*r*r/5}" ixy="0" ixz="0" iyy="${2*m*r*r/5}" iyz="0" izz="${2*m*r*r/5}"/>
   </xacro:macro>
