Commit message: Add ouster & refactor

File: urdf/OS1-64.urdf.xacro (robot description, xacro)
@@ -24,5 +24,5 @@
          <origin xyz="0 0 0.0" rpy="0 0 1.5707" />
          <geometry>
-	         <mesh filename="package://ouster_description/meshes/os1_64.dae" />
+	         <mesh filename="package://rover_description/meshes/os1_64.dae" />
            <!-- <cylinder length="0.073" radius="0.04" /> -->
          </geometry>

File: urdf/rover1.urdf.xacro (robot description, xacro)
@@ -1,5 +1,6 @@
 <?xml version="1.0"?>
-<robot name="rover" xmlns:xacro="http://www.ros.org/wiki/xacro">
+<robot xmlns:xacro="http://www.ros.org/wiki/xacro" name="rover">
   <xacro:property name="PI" value="3.1415926535897931" />
+<!--############ ROBOT PROPERTIES ENSURE THIS IS UP TO DATE #################-->
   <xacro:property name="wheelbase" value="0.262" />
   <xacro:property name="track" value="0.37559" />
@@ -13,10 +14,45 @@
   <xacro:property name="dummy_inertia" value="1e-09"/>
   <xacro:property name="mount_spacing" value="0.120" />
+<!--###################################################-->
   <material name="dark_grey"><color rgba="0.2 0.2 0.2 1.0" /></material>
   <material name="light_grey"><color rgba="0.4 0.4 0.4 1.0" /></material>
   <material name="yellow"><color rgba="0.8 0.8 0.0 1.0" /></material>
   <material name="black"><color rgba="0.15 0.15 0.15 1.0" /></material>
+  <material name="blue"><color rgba="0 0 0.8 1"/></material>
+  <!-- Base Footprint -->
+  <link name="base_footprint" />
+  <!-- Base Link -->
+  <joint name="footprint" type="fixed" >
+   <parent link="base_footprint" />
+    <child link="base_link" />
+    <origin xyz="0 0 0.05" rpy="0 0 0" />
+  </joint>
+  <link name="base_link" >
+  <origin xyz="0 0 ${footprint_vertical_offset}" rpy="${PI/2} 0 ${PI/2}"/>
+    <visual>
+      <geometry>
+        <box size="${chassis_length} ${chassis_width} ${chassis_height}" />
+      </geometry>
+    </visual>
+    <collision>
+      <geometry>
+        <box size="${chassis_length} ${chassis_width} ${chassis_height}" />
+      </geometry>
+    </collision>
+    <inertial>
+      <origin xyz="0 0 0"/>
+      <mass value="10"/>
+      <inertia ixx="3.0" ixy="0.0" ixz="0.0"
+               iyy="3.0" iyz="0.0"
+               izz="3.0" />
+    </inertial>
+  </link>
+  <!-- Bug fix: changed type from continuous to fixed to get rid of a bug
+  https://www.reddit.com/r/ROS/comments/e3u3ru/rviz_error_no_transform_from_wheel_left_link/-->
+  <!-- use xacro macros to improve readability and make it simpler refer to:
+  http://library.isr.ist.utl.pt/docs/roswiki/xacro.html
+  https://github.com/jackal/jackal/blob/46baf37703fcee690d1d85dfc2bb9153abc38fbe/jackal_description/urdf/jackal.urdf.xacro#L26-L93-->
   <xacro:macro name="wheel" params="prefix *joint_pose">
-    <link name="${prefix}_wheel_link">
+       <link name="${prefix}_wheel_link">
       <visual>
         <origin xyz="0 0 0" rpy="${PI/2} 0 0"/>
@@ -42,23 +78,21 @@
     </link>
     <gazebo reference="${prefix}_wheel_link">
-      <material>Gazebo/DarkGrey</material>
-      <selfCollide>false</selfCollide>
-      <mu1 value="0.5"/>
-      <mu2 value="0.5"/>
-      <kp value="10000000.0" />
-      <kd value="1" />
-      <fdir1 value="1 0 0"/>
+        <material>Gazebo/DarkGrey</material>
+        <selfCollide>false</selfCollide>
+        <mu1 value="0.5"/>
+        <mu2 value="0.5"/>
+        <kp value="10000000.0" />
+        <kd value="1" />
+        <fdir1 value="1 0 0"/>
     </gazebo>
-    <joint name="${prefix}_wheel" type="continuous">
-      <parent link="chassis_link"/>
-      <child link="${prefix}_wheel_link" />
-      <xacro:insert_block name="joint_pose" />
-      <axis xyz="0 1 0" />
+    <joint name="${prefix}_wheel_hinge" type="continuous">
+      <parent link="base_link"/>
+      <child link="${prefix}_wheel_link"/>
+      <axis xyz="0 1 0"/>
+      <origin xyz="0 0 0"/>
     </joint>
-    <!-- In reality, Jackal has only two motors, one per side. However, it's more
-         straightforward for Gazebo to simulate as if there's an actuator per wheel. -->
     <transmission name="${prefix}_wheel_trans">
       <type>transmission_interface/SimpleTransmission</type>
-      <joint name="${prefix}_wheel">
+      <joint name="${prefix}_wheel_hinge">
         <hardwareInterface>hardware_interface/VelocityJointInterface</hardwareInterface>
       </joint>
@@ -74,46 +108,25 @@
     <origin xyz="${wheelbase/2} ${-track/2} ${wheel_vertical_offset}" rpy="0 0 0" />
   </xacro:wheel>
-  <xacro:wheel prefix="rear_left">
+  <xacro:wheel prefix="back_left">
     <origin xyz="${-wheelbase/2} ${track/2} ${wheel_vertical_offset}" rpy="0 0 0" />
   </xacro:wheel>
-  <xacro:wheel prefix="rear_right">
+  <xacro:wheel prefix="back_right">
     <origin xyz="${-wheelbase/2} ${-track/2} ${wheel_vertical_offset}" rpy="0 0 0" />
   </xacro:wheel>
-  <link name="base_link"></link>
-  <joint name="base_link_joint" type="fixed">
-    <origin xyz="0 0 0" rpy="0 0 0" />
-    <parent link="base_link"/>
-    <child link="chassis_link" />
-  </joint>
-  <link name="chassis_link">
-    <visual>
-      <origin xyz="0 0 ${footprint_vertical_offset}" rpy="${PI/2} 0 0"/>
-      <geometry>
-        <box size="${chassis_length} ${chassis_width} ${chassis_height}"/>
-      </geometry>
-      <material name="dark_grey" />
-    </visual>
-    <collision>
-      <origin xyz="0 0 ${chassis_height/2}"/>
-      <geometry>
-        <box size="${chassis_length} ${chassis_width} ${chassis_height}"/>
-      </geometry>
-    </collision>
-    <inertial>
-      <!-- Center of mass -->
-      <origin xyz="0.012  0.002 0.067" rpy="0 0 0"/>
-      <mass value="16.523"/>
-      <!-- Moments of inertia: ( chassis without wheels ) -->
-      <inertia
-        ixx="0.3136" ixy="-0.0008" ixz="0.0164"
-        iyy="0.3922" iyz="-0.0009"
-        izz="0.4485"/>
-      </inertial>
-  </link>
   <xacro:include filename="$(find rover_description)/urdf/OS1-64.urdf.xacro"/>
   <xacro:OS1-64 parent="base_link" name="os1_sensor" hz="10" samples="220">
     <origin xyz="${chassis_length} ${chassis_width} ${chassis_height}" rpy="$0 0 0" />
   </xacro:OS1-64>
-  <!-- Bring in simulation data for Gazebo. -->
+  <link name="imu_link">
+    <inertial>
+      <mass value="0.001"/>
+      <origin xyz="0 0 0" rpy="0 0 0"/>
+      <inertia ixx="${dummy_inertia}" ixy="0.0" ixz="0.0" iyy="${dummy_inertia}" iyz="0.0" izz="${dummy_inertia}"/>
+    </inertial>
+  </link>
+  <joint name="imu_joint" type="fixed">
+    <parent link="base_link" /> <!--TODO: check base_link or base_footprint-->
+    <child link="imu_link" />
+  </joint>
   <xacro:include filename="$(find rover_description)/urdf/rover.gazebo" />
 </robot>
