Commit message: Changed the length and width of the base

File: urdf/rover.urdf.xacro (robot description, xacro)
@@ -3,6 +3,6 @@
   <xacro:property name="PI" value="3.1415926535897931"/>
   <xacro:property name="chassisHeight" value="0.3"/>
-  <xacro:property name="chassisLength" value="0.75"/>
-  <xacro:property name="chassisWidth" value="0.45"/>
+  <xacro:property name="chassisLength" value="0.9"/>
+  <xacro:property name="chassisWidth" value="0.6"/>
   <xacro:property name="chassisMass" value="10"/>
   <xacro:property name="wheelWidth" value="0.075"/>

Commit message: Model now works with ouster lidar

File: urdf/rover.urdf.xacro (robot description, xacro)
@@ -111,9 +111,9 @@
       </inertial>
   </link>
-  <xacro:include filename="$(find rover_description)/urdf/OS1-64.urdf.xacro"/>
-  <xacro:OS1-64 parent="base_link" name="os1_sensor" hz="10" samples="220">
-    <origin xyz="${chassis_length} ${chassis_width} ${chassis_height}" rpy="$0 0 0" />
-  </xacro:OS1-64>
   <!-- Bring in simulation data for Gazebo. -->
   <xacro:include filename="$(find rover_description)/urdf/rover.gazebo" />
+  <xacro:include filename="$(find rover_description)/urdf/OS1-64.urdf.xacro"/>
+  <xacro:OS1-64 parent="chassis_link" name="os1_sensor" hz="10" samples="220">
+    <origin xyz="0 0 ${chassis_height}" rpy="0 0 0" />
+  </xacro:OS1-64>
 </robot>
